File: Projeto Base/Projeto-Natal-2023-Base/Projeto-Natal-2023-Base.kicad_pcb (KiCad board)
At the start: 2 copper layers, 39 parts, among them J1 Conn_01x03_Pin, U1 CH32V003F4P6

Commit message: Draft 1
Parts:
- removed D1, D2, D3, D4: LED R, LED_THT:LED_D5.0mm
- removed D10, D11, D12, D9: LED B, LED_THT:LED_D5.0mm
- removed D13, D14, D15, D16: LED Y, LED_THT:LED_D5.0mm
- removed D5, D6, D7, D8: LED G, LED_THT:LED_D5.0mm
- added REF**: MountingHole_3.2mm_M3, MountingHole:MountingHole_3.2mm_M3, F.Cu at (94.0, 76.8)
- BT1: moved to B.Cu
- moved C2 84.0 mm to (87.9, 103.5), turned to 180 degrees
- moved C3 82.2 mm to (88.0, 101.6)
- moved U1 72.4 mm to (93.7, 99.4)
- moved R1 71.5 mm to (88.0, 99.7)
- moved C1 71.4 mm to (88.0, 97.8)
- moved BT1 57.1 mm to (94.0, 99.1), turned to 180 degrees
- moved R11 2.77 mm to (168.6, 127.0)
Other:
- board outline added: 50 x 50 mm

Commit message: update
Parts:
- moved C2 6.39 mm to (94.0, 105.4)
- moved C3 6.11 mm to (93.9, 103.4)
- moved U1 0.75 mm to (93.9, 98.7)
Changed lines of the file:
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@@
   )
   (footprint "Capacitor_SMD:C_0603_1608Metric_Pad1.08x0.95mm_HandSolder" (layer "F.Cu")
-    (at 88.0375 101.6)
+    (at 93.8795 103.378)
     (descr "Capacitor SMD 0603 (1608 Metric), square (rectangular) end terminal, IPC_7351 nominal with elongated pad for handsoldering. (Body size source: IPC-SM-782 page 76, https://www.pcb-3d.com/wordpress/wp-content/uploads/ipc-sm-782a_amendment_1_and_2.pdf), generated with kicad-footprint-generator")
     (tags "capacitor handsolder")
@@
   )
   (footprint "Package_SO:TSSOP-20_4.4x6.5mm_P0.65mm" (layer "F.Cu")
-    (at 93.6675 99.415)
+    (at 93.9115 98.705)
     (descr "TSSOP, 20 Pin (JEDEC MO-153 Var AC https://www.jedec.org/document_search?search_api_views_fulltext=MO-153), generated with kicad-footprint-generator ipc_gullwing_generator.py")
     (tags "TSSOP SO")
@@
   )
   (footprint "Capacitor_SMD:C_0805_2012Metric_Pad1.18x1.45mm_HandSolder" (layer "F.Cu")
-    (at 87.8625 103.505 180)
+    (at 93.9585 105.41 180)
     (descr "Capacitor SMD 0805 (2012 Metric), square (rectangular) end terminal, IPC_7351 nominal with elongated pad for handsoldering. (Body size source: IPC-SM-782 page 76, https://www.pcb-3d.com/wordpress/wp-content/uploads/ipc-sm-782a_amendment_1_and_2.pdf, https://docs.google.com/spreadsheets/d/1BsfQQcO9C6DZCsRaXUlFlo91Tg2WpOkGARC1WS5S8t0/edit?usp=sharing), generated with kicad-footprint-generator")
     (tags "capacitor handsolder")

Commit message: posicionando os componentes
Parts:
- removed R14, R15, R16, R17: 1K, Resistor_SMD:R_0603_1608Metric_Pad0.98x0.95mm_HandSolder
- added D1: LED, LED_SMD:LED_0805_2012Metric, F.Cu at (89.4, 76.5)
- added D10: LED, LED_SMD:LED_0805_2012Metric, F.Cu at (72.9, 107.8)
- added D11: LED, LED_SMD:LED_0805_2012Metric, F.Cu at (75.0, 111.9)
- added D12: LED, LED_SMD:LED_0805_2012Metric, F.Cu at (77.9, 115.2)
- added D13: LED, LED_SMD:LED_0805_2012Metric, F.Cu at (81.4, 118.1)
- added D14: LED, LED_SMD:LED_0805_2012Metric, F.Cu at (85.5, 120.3)
- added D15: LED, LED_SMD:LED_0805_2012Metric, F.Cu at (89.4, 121.4)
- added D16: LED, LED_SMD:LED_0805_2012Metric, F.Cu at (98.6, 121.5)
- added D17: LED, LED_SMD:LED_0805_2012Metric, F.Cu at (102.7, 120.3)
- added D18: LED, LED_SMD:LED_0805_2012Metric, F.Cu at (106.8, 118.0)
- added D19: LED, LED_SMD:LED_0805_2012Metric, F.Cu at (110.2, 115.2)
- added D2: LED, LED_SMD:LED_0805_2012Metric, F.Cu at (85.2, 77.8)
- added D20: LED, LED_SMD:LED_0805_2012Metric, F.Cu at (113.1, 111.7)
- added D21: LED, LED_SMD:LED_0805_2012Metric, F.Cu at (115.2, 107.8)
- added D22: LED, LED_SMD:LED_0805_2012Metric, F.Cu at (116.5, 103.8)
- added D23: LED, LED_SMD:LED_0805_2012Metric, F.Cu at (117.0, 99.1)
- added D24: LED, LED_SMD:LED_0805_2012Metric, F.Cu at (116.5, 94.5)
- added D25: LED, LED_SMD:LED_0805_2012Metric, F.Cu at (115.3, 90.3)
- added D26: LED, LED_SMD:LED_0805_2012Metric, F.Cu at (113.3, 86.4)
- added D27: LED, LED_SMD:LED_0805_2012Metric, F.Cu at (110.2, 82.8)
- added D28: LED, LED_SMD:LED_0805_2012Metric, F.Cu at (106.8, 80.0)
- added D29: LED, LED_SMD:LED_0805_2012Metric, F.Cu at (102.6, 77.7)
- added D3: LED, LED_SMD:LED_0805_2012Metric, F.Cu at (81.5, 79.8)
- added D30: LED, LED_SMD:LED_0805_2012Metric, F.Cu at (98.6, 76.6)
- added D4: LED, LED_SMD:LED_0805_2012Metric, F.Cu at (77.7, 82.8)
- added D5: LED, LED_SMD:LED_0805_2012Metric, F.Cu at (74.9, 86.4)
- added D6: LED, LED_SMD:LED_0805_2012Metric, F.Cu at (72.7, 90.5)
- added D7: LED, LED_SMD:LED_0805_2012Metric, F.Cu at (71.6, 94.4)
- added D8: LED, LED_SMD:LED_0805_2012Metric, F.Cu at (71.1, 99.1)
- added D9: LED, LED_SMD:LED_0805_2012Metric, F.Cu at (71.6, 103.6)
- added Q1: BC817, Package_TO_SOT_SMD:SOT-23, F.Cu at (94.2, 83.8)
- added Q2: BC817, Package_TO_SOT_SMD:SOT-23, F.Cu at (94.2, 88.2)
- added Q3: BC817, Package_TO_SOT_SMD:SOT-23, F.Cu at (94.2, 111.1)
- added Q4: BC817, Package_TO_SOT_SMD:SOT-23, F.Cu at (94.2, 115.5)
- moved R11 87.8 mm to (88.0, 92.1)
- moved R10 86.2 mm to (88.0, 90.3)
- moved R13 84.4 mm to (88.0, 95.5)
- moved R12 81.1 mm to (88.0, 93.7)
- moved J1 79.4 mm to (102.2, 110.8), turned to 135 degrees
- moved R9 67.7 mm to (100.6, 93.6)
- moved R8 67.5 mm to (100.6, 95.1)
- moved R7 64.0 mm to (100.6, 96.6)
- moved R3 63.5 mm to (100.6, 102.7)
- moved R6 63.4 mm to (100.6, 98.2)
- moved R4 63.2 mm to (100.6, 101.2)
- moved R5 63.2 mm to (100.6, 99.7)
- moved R2 58.9 mm to (100.6, 104.3)
- moved REF** 0.84 mm to (94.0, 76.0)
Connections:
- R10 pad 1: Net-(U1-PC0) -> C1
- R10 pad 2: LED11 -> Net-(Q1-B)
- R11 pad 1: Net-(U1-PC1) -> C2
- R11 pad 2: LED11 -> Net-(Q2-B)
- R12 pad 1: Net-(U1-PC2) -> C3
- R12 pad 2: LED11 -> Net-(Q3-B)
- R13 pad 1: Net-(U1-PC3) -> C4
- R13 pad 2: LED12 -> Net-(Q4-B)
- R2 pad 1: LED1 -> Net-(U1-PC0)
- R2 pad 2: Net-(U1-OSC_IN/PA1) -> L1
- R3 pad 1: LED2 -> Net-(U1-PC1)
- R3 pad 2: Net-(U1-OSC_OUT/PA2) -> L2
- R4 pad 1: LED3 -> Net-(U1-PC2)
- R4 pad 2: Net-(U1-PD0) -> L3
- R5 pad 1: LED4 -> Net-(U1-PC3)
- R5 pad 2: Net-(U1-PD2) -> L4
- R6 pad 1: LED5 -> Net-(U1-PC4)
- R6 pad 2: Net-(U1-PD3) -> L5
- R7 pad 1: LED6 -> Net-(U1-PC5)
- R7 pad 2: Net-(U1-PD4) -> L6
- R8 pad 1: LED7 -> Net-(U1-PC6)
- R8 pad 2: Net-(U1-PD5) -> L7
- R9 pad 1: LED8 -> Net-(U1-PC7)
- R9 pad 2: Net-(U1-PD6) -> L8
- U1 pad 1: Net-(U1-PD4) -> C2
- U1 pad 19: Net-(U1-PD2) -> unconnected-(U1-PD2-Pad19)
- U1 pad 2: Net-(U1-PD5) -> C3
- U1 pad 20: Net-(U1-PD3) -> C1
- U1 pad 3: Net-(U1-PD6) -> C4
- U1 pad 5: Net-(U1-OSC_IN/PA1) -> unconnected-(U1-OSC_IN/PA1-Pad5)
- U1 pad 6: Net-(U1-OSC_OUT/PA2) -> unconnected-(U1-OSC_OUT/PA2-Pad6)
- U1 pad 8: Net-(U1-PD0) -> unconnected-(U1-PD0-Pad8)

Commit message: routing...
Parts:
- moved Q4 24.4 mm to (111.1, 98.0)
- moved Q1 22.2 mm to (77.1, 98.0), turned to 180 degrees
- moved Q2 22.0 mm to (77.1, 102.0), turned to 180 degrees
- moved R12 21.6 mm to (108.0, 101.9), turned to 90 degrees
- moved R13 20.1 mm to (108.0, 97.9), turned to 90 degrees
- moved Q3 19.2 mm to (111.1, 102.0)
- moved R11 12.7 mm to (80.0, 101.9), turned to -90 degrees
- moved R10 11.0 mm to (80.0, 97.9), turned to -90 degrees
- moved J1 10.5 mm to (92.0, 113.0), turned to 90 degrees
- moved C2 6.33 mm to (88.2, 102.9)
- moved C3 6.04 mm to (88.3, 101.1)
- moved R2 1.76 mm to (102.1, 105.2)
- moved R3 1.76 mm to (102.1, 103.6)
- moved R4 1.76 mm to (102.1, 102.1)
- moved R5 1.76 mm to (102.1, 100.6)
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Connections:
- D16 pad 1: Net-(D10-K) -> Net-(D16-K)
- D16 pad 2: L8 -> L7
- D17 pad 1: Net-(D17-K) -> Net-(D16-K)
- D17 pad 2: L1 -> L6
- D18 pad 1: Net-(D17-K) -> Net-(D16-K)
- D18 pad 2: L2 -> L5
- D19 pad 1: Net-(D17-K) -> Net-(D16-K)
- D19 pad 2: L3 -> L4
- D20 pad 1: Net-(D17-K) -> Net-(D16-K)
- D20 pad 2: L4 -> L3
- D21 pad 1: Net-(D17-K) -> Net-(D16-K)
- D21 pad 2: L5 -> L2
- D22 pad 1: Net-(D17-K) -> Net-(D16-K)
- D22 pad 2: L6 -> L1
- D23 pad 1: Net-(D17-K) -> Net-(D23-K)
- D23 pad 2: L7 -> L8
- D24 pad 1: Net-(D17-K) -> Net-(D23-K)
- D24 pad 2: L8 -> L7
- D25 pad 1: Net-(D25-K) -> Net-(D23-K)
- D25 pad 2: L1 -> L6
- D26 pad 1: Net-(D25-K) -> Net-(D23-K)
- D26 pad 2: L2 -> L5
- D27 pad 1: Net-(D25-K) -> Net-(D23-K)
- D27 pad 2: L3 -> L4
- D28 pad 1: Net-(D25-K) -> Net-(D23-K)
- D28 pad 2: L4 -> L3
- D29 pad 1: Net-(D25-K) -> Net-(D23-K)
- D29 pad 2: L5 -> L2
- D30 pad 1: Net-(D25-K) -> Net-(D23-K)
- D30 pad 2: L6 -> L1
- Q3 pad 3: Net-(D17-K) -> Net-(D16-K)
- Q4 pad 3: Net-(D25-K) -> Net-(D23-K)
Routing:
- net L4: track 0.00 -> 85.0 mm, vias 0 -> 2
- net L5: track 0.00 -> 80.3 mm, vias 0 -> 2
- net L3: track 0.00 -> 77.9 mm, vias 0 -> 2
- net L6: track 0.00 -> 73.7 mm, vias 0 -> 2
- net L2: track 0.00 -> 70.2 mm, vias 0 -> 2
- net L7: track 0.00 -> 66.6 mm, vias 0 -> 2
- net L1: track 0.00 -> 63.0 mm
- net L8: track 0.00 -> 55.6 mm
- net C2: track 0.00 -> 13.2 mm
- net Net-(U1-PC0): track 0.00 -> 11.4 mm
- net +3V3: track 0.00 -> 6.63 mm
- net Net-(U1-PC1): track 0.00 -> 5.86 mm
- net Net-(U1-PC7): track 0.00 -> 5.79 mm
- net Net-(U1-PC6): track 0.00 -> 5.43 mm
- net Net-(U1-PC5): track 0.00 -> 5.07 mm
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
Commit message: v1.0.0
Parts:
- added BZ1: Buzzer, Library:PassiveBuzzerSMD_JiangsuHuaneng_MLT-5030, B.Cu at (92.7, 83.2)
- added J2: Conn_01x01_Pin, TestPoint:TestPoint_Pad_D2.0mm, B.Cu at (110.5, 85.7)
- added J3: Conn_01x01_Pin, TestPoint:TestPoint_Pad_D2.0mm, B.Cu at (110.5, 88.3)
- added J4: Conn_01x01_Pin, TestPoint:TestPoint_Pad_D2.0mm, B.Cu at (110.5, 90.8)
- added Q5: MMBT3906, Package_TO_SOT_SMD:SOT-23, B.Cu at (94.0, 87.7)
- added R14: 1K, Resistor_SMD:R_0603_1608Metric_Pad0.98x0.95mm_HandSolder, B.Cu at (90.8, 87.6)
- added SW1: SW_Push, Button_Switch_SMD:SW_Push_1P1T_NO_6x6mm_H9.5mm, B.Cu at (100.3, 85.7)
- BT1: footprint Battery:BatteryHolder_Keystone_3002_1x2032 -> Battery:BatteryHolder_Multicomp_BC-2001_1x2032
- C1, C2, C3, Q1, Q2, Q3, Q4, R1, R10, R11, R12, R13, R2, R3, R4, R5, R6, R7, R8, R9, U1: moved to B.Cu
- J1: value Conn_01x03_Pin -> Conn_01x01_Pin; footprint Connector_PinHeader_2.54mm:PinHeader_1x03_P2.54mm_Vertical -> TestPoint:TestPoint_Pad_D2.0mm; moved to B.Cu
- moved J1 27.0 mm to (110.5, 93.3), turned to -135 degrees
- moved R5 16.2 mm to (86.2, 97.5), turned to 180 degrees
- moved R6 16.2 mm to (86.2, 96.0), turned to 180 degrees
- moved R7 16.2 mm to (86.2, 94.5), turned to 180 degrees
- moved R8 16.2 mm to (86.2, 93.0), turned to 180 degrees
- moved R9 16.2 mm to (86.2, 91.4), turned to 180 degrees
- moved R2 16.2 mm to (86.2, 102.1), turned to 180 degrees
- moved R3 16.2 mm to (86.2, 100.6), turned to 180 degrees
- moved R4 16.2 mm to (86.2, 99.1), turned to 180 degrees
- moved Q1 13.8 mm to (86.3, 87.6)
- moved C2 13.8 mm to (101.2, 98.4), turned to 0 degrees
- moved R10 13.7 mm to (89.0, 87.6), turned to 90 degrees
- moved C1 13.6 mm to (101.1, 93.6), turned to 180 degrees
- moved R1 13.6 mm to (101.1, 95.1), turned to 180 degrees
- moved C3 13.6 mm to (101.1, 96.6)
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Connections:
- J1 pad 1: +3V3 -> unconnected-(J1-Pin_1-Pad1)
- U1 pad 19: unconnected-(U1-PD2-Pad19) -> BZR
- U1 pad 8: unconnected-(U1-PD0-Pad8) -> BT
Routing:
- net +3V3: track 6.63 -> 103.2 mm, vias 0 -> 3
- net Net-(D1-K): track 0.27 -> 54.6 mm, vias 0 -> 1
- net Net-(D23-K): track 0.98 -> 47.7 mm, vias 0 -> 1
- net Net-(D10-K): track 0.93 -> 45.1 mm, vias 0 -> 1
- net L6: track 73.7 -> 116.8 mm, vias 2 -> 6
- net Net-(D16-K): track 0.00 -> 38.5 mm, vias 0 -> 1
- net C2: track 13.2 -> 49.4 mm, vias 0 -> 2
- net L5: track 80.3 -> 114.9 mm, vias 2 -> 6
- net L2: track 70.2 -> 104.0 mm, vias 2 -> 5
- net L1: track 63.0 -> 94.8 mm, vias 0 -> 4
- net L4: track 85.0 -> 115.1 mm, vias 2 -> 6
- net L3: track 77.9 -> 107.9 mm, vias 2 -> 5
- net L7: track 66.6 -> 93.4 mm, vias 2 -> 3
- net C3: track 0.00 -> 23.5 mm
- net SWIO: track 0.00 -> 23.2 mm, vias 0 -> 2
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- added copper zone on B.Cu, net GND
- added copper zone on F.Cu, net GND
Other:
- board text added: "3V3"
- board text added: "GND"
- board text added: "NC"
- board text added: "SWIO"
