File: Projeto Base/Projeto-Natal-2023-Base/Projeto-Natal-2023-Base.kicad_pcb (KiCad board)
At the start: 2 copper layers, 50 x 50 mm, 61 parts, among them J1 Conn_01x01_Pin, J2 Conn_01x01_Pin, J3 Conn_01x01_Pin, J4 Conn_01x01_Pin, Q1 BC817, Q2 BC817, Q3 BC817, Q4 BC817, Q5 MMBT3906, SW1 SW_Push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

Commit message: Versão para revisão
Parts:
- added G***: LOGO, Library:natal-franzininho, F.Cu at (94.0, 98.8)
- added G***: LOGO, Library:logoFranzininho_15x15, B.Cu at (78.8, 90.1)
Routing:
- net L7: track 93.4 -> 91.5 mm
- net GND: vias 8 -> 15
Other:
- board text added: "Christmas Ball"
- board text added: "Feliz Natal!"
- board text added: "Projeto Natal 2023"
- board text added: "REV 1.0.0"
- board text added: "by Fábio Souza"
