File: Projeto Base/Projeto-Natal-2023-Base/_autosave-Projeto-Natal-2023-Base.kicad_pcb (KiCad board)
At the start: 2 copper layers, 77.8 x 77.8 mm, 71 parts, among them J1 Conn_01x01_Pin, J2 Conn_01x01_Pin, J3 Conn_01x01_Pin, J4 Conn_01x01_Pin, J5 Conn_01x01_Pin, J6 Conn_01x01_Pin, J7 Conn_01x01_Pin, J8 Conn_01x01_Pin, Q1 BC817, Q2 BC817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

Commit message: V1.1.0
Placa com 78,8 mm de diametro
Parts:
- D1, D10, D13, D18, D21, D24, D27, D30, D4, D7: value LED -> D-B080508B1-KS2
- D11, D14, D17, D2, D20, D23, D26, D29, D5, D8: value LED -> e17-21SURC/S530-A3/TR8
- D12, D15, D16, D19, D22, D25, D28, D3, D6, D9: value LED -> NCD0805G1
